File: Lab7/problem2/problem2.kicad_pcb (KiCad board)
At the start: 2 copper layers, 27.9 x 35.6 mm, 10 parts, among them J1 Conn_01x02_Male, U1 NE555D

Commit message: Lab8
Routing:
- net /pin_7: track 42.3 -> 41.5 mm
